Commit message: commit2

File: description/example_robot.urdf.xacro (robot description, xacro)
@@ -88,5 +88,5 @@
     <!-- - The visual/collision origin is set to halfway along the length (similar to the box), but also with a rotation (again using the mathematical features). -->
     <!--   This is because the cylinder extends along the Z axis by default, but we want it to be along the X axis (when the joint is at 0) -->
-    <xacro:property name="arm_length" value="2" />
+    <xacro:property name="arm_length" value="3" />
     <xacro:property name="arm_radius" value="0.04" />
     <link name="arm_link">
